File: Electronics/EspressoCircuitry/EspressoCircuitry.sch (EAGLE design)
At the start: 73 parts, among them IC1 TB6612FNG, IC2 TB6612FNG, IC3 TB6612FNG, J1 1X2-3.5MM, J10 1X2-3.5MM, J11 1X2-3.5MM, J12 1X2-3.5MM, J13 1X2-3.5MM, J14 1X2-3.5MM, J15 1X2-3.5MM, J16 1X2-3.5MM, J17 1X2-3.5MM, J18 1X2-3.5MM, J19 1X2-3.5MM, J2 1X2-3.5MM, J20 1X2-3.5MM, J21 1X2-3.5MM, J22 1X2-3.5MM, J23 1X2-3.5MM, J3 1X2-3.5MM, J4 1X2-3.5MM, J5 1X2-3.5MM, J6 1X2-3.5MM, J7 1X2-3.5MM, J8 1X2-3.5MM, J9 1X2-3.5MM, K1 G5LE, K2 G5LE, K3 G5LE, K4 G5LE

Commit message: Added updated PCB files
Parts:
- removed C20, C21, C22, C23: 10u, rcl:CPOL-USE2.5-5
- added IC4: REG1117, burr-brown:REG1117
- added J24, J25, J26, J27, J28: 1X2-3.5MM, adafruit:1X2-3.5MM
- added JP1, JP2, JP3, JP4: (no value), adafruit:PINHD-1X3
- added R11: 10k, rcl:R-US_R0603
- added SJ1, SJ10, SJ11, SJ12, SJ2, SJ3, SJ4, SJ5, SJ6, SJ7, SJ8, SJ9: (no value), jumper:SJ
- C24, C25: value 10u -> 100u
Connections:
- removed net SWCLK: SV1.2
- new net FLOW1: J25.2, U$2.PB12
- new net FLOW2: J27.2, U$2.PB2
- new net GROUND_SENSE: J24.2, R11.2, U$2.PA0
- new net N$44: JP1.2, SJ1.2, SJ2.2
- new net N$45: JP2.2, SJ3.2, SJ4.2
- new net N$46: JP3.2, SJ5.2, SJ6.2
- new net N$47: JP4.2, SJ7.2, SJ8.2
- new net N$48: SJ11.1, SJ12.1, U$1.RX
- new net SERVO1: JP1.1, U$2.PC6
- new net SERVO2: JP2.1, U$2.PC7
- new net SERVO3: JP3.1, U$2.PC8
- new net SERVO4: JP4.1, U$2.PC9
- net +12V: now also IC4.VIN; no longer C21.+, C23.+
- net +3V3: now also C13.1, IC4.VOUT, J24.1, SJ1.1, SJ3.1, SJ5.1, SJ7.1; no longer C20.+, C22.+
- net +5V: now also J25.1, J27.1, SJ2.1, SJ4.1, SJ6.1, SJ8.1
- net GND: now also C18.2, IC4.GND, J26.1, J26.2, J28.1, J28.2, JP1.3, JP2.3, JP3.3, JP4.3, R11.1; no longer C20.-, C21.-, C22.-, C23.-
- net M1_AIN1: now also U$2.PB3
- net M1_AIN2: now also U$2.PB4
- net M1_BIN1: now also U$2.PB5
- net M1_BIN2: now also U$2.PB6
- net M1_PWMA: now also U$2.PA8
- net M1_PWMB: now also U$2.PA9
- net M2_AIN1: now also U$2.PB7
- net M2_AIN2: now also U$2.PC0
- net M2_BIN1: now also U$2.PC1
- net M2_BIN2: now also U$2.PC2
- net M2_PWMA: now also U$2.PA10
- net M2_PWMB: now also U$2.PA11
- net M3_AIN1: now also U$2.PC3
- net M3_AIN2: now also U$2.PA6
- net M3_BIN1: now also U$2.PA7
- net M3_BIN2: now also U$2.PB0
- net M3_PWMA: now also U$2.PB10
- net M3_PWMB: now also U$2.PB11
- net N$1: now also SJ10.1, SJ9.1, U$1.TX; no longer U$2.PA4
- net PRESSURE1: now also U$2.PA4
- net PRESSURE2: now also U$2.PA5
- net RX: now also SJ11.2, SJ9.2; no longer U$1.TX
- net SWDCLK: now also SV1.2
- net TEMP1: now also U$2.PA1
- net TEMP2: now also U$2.PA2
- net TEMP3: now also U$2.PA3
- net TX: now also SJ10.2, SJ12.2; no longer U$1.RX
- net ~RELAY1: now also U$2.PC10
- net ~RELAY2: now also U$2.PC11
- net ~RELAY3: now also U$2.PC12
- net ~RELAY4: now also U$2.PD2
Other:
- note added: "ADC_IN4"
- note added: "ADC_IN5"
- note added: "AF0"
- note added: "AF2"
- note added: "EXTI1 and EXTI2"
- note added: "J1"
- note added: "J10"
- note added: "J11"
- note added: "J12"
- note added: "J13"
- note added: "J14"
- note added: "J15"
- note added: "J16"
- note added: "J17"
- note added: "J18"
- note added: "J19"
- note added: "J2"
- note added: "J20"
- note added: "J21"
- note added: "J22"
- note added: "J23"
- note added: "J3"
- note added: "J4"
- note added: "J5"
- note added: "J6"
- note added: "J7"
- note added: "J8"
- note added: "J9"
- note added: "PA0-PA3 -> ADC_IN0-ADC_IN3"
- note added: "PA8-PA11 -> TIM1_CH1 - TIM1_CH4"
- note added: "PB10 -> TIM2_CH3 PB11 -> TIM3_CH4"
- note added: "PC6 - PC9 -> TIM3_CH1 - TIM3_CH4"
- moved on the sheet: C19, C24, C25, IC1, IC2, IC3, R4, R5, R6
